File: Hardware/SimpleControllboard/SimpleControllboard.sch (EAGLE design)
At the start: 14 parts, among them IC4 ATmega328P, Q2 FDD4141TO252, Y2 16MHz

Commit message: New PCBs
Parts:
- removed C2: 0.1uF, microbuilder:CAP_CERAMIC0805-NOOUTLINE
- removed JP2, JP3, JP4, JP5, JP6: (no value), pinhead:PINHD-2X3
- removed JP7: (no value), pinhead:PINHD-1X4
- added C1: 0.1uF, microbuilder:CAP_CERAMIC0805-NOOUTLINE
- added U$1: AKZ692-10, HeRo:AKZ692-10
- added U$3: AKZ692-2, HeRo:AKZ692-2
- JP1: device pinhead:PINHD-2X3 -> pinhead:PINHD-1X4
- U$2: value AKZ692-5 -> AKZ692-10; device HeRo:AKZ692-5 -> HeRo:AKZ692-10
Connections:
- removed net A6: IC4.ADC6
- removed net A7: IC4.ADC7
- removed net RXD: IC4.PD0(RXD), JP7.2
- removed net SCL: IC4.PC5(ADC5/SCL), U$2.5
- removed net SDA: IC4.PC4(ADC4/SDA), U$2.4
- removed net TXD: IC4.PD1(TXD), JP7.1
- new net A4: IC4.PC4(ADC4/SDA), U$1.2
- new net A5: IC4.PC5(ADC5/SCL), U$1.1
- new net D0: IC4.PD0(RXD), JP1.2, U$2.1
- new net D1: IC4.PD1(TXD), JP1.1, U$2.2
- net +5V: no longer JP1.3, JP1.4, JP2.3, JP2.4, JP3.3, JP3.4, JP4.3, JP4.4, JP5.3, JP5.4, JP6.3, JP6.4
- net A0: now also U$1.6; no longer JP4.2
- net A1: now also U$1.5; no longer JP5.2
- net A2: now also U$1.4; no longer JP6.1
- net A3: now also U$1.3; no longer JP6.2
- net D10: now also U$1.10; no longer JP1.2
- net D11: now also U$1.9; no longer JP2.1
- net D12: now also U$1.8; no longer JP2.2
- net D13: now also U$1.7; no longer JP3.1
- net D2: now also U$2.3
- net D3: now also U$2.4
- net D4: now also U$2.5; no longer JP5.1
- net D5: now also U$2.6; no longer JP4.1
- net D6: now also U$2.7; no longer JP3.2
- net D7: now also U$2.8
- net D8: now also U$2.9
- net D9: now also U$2.10; no longer JP1.1
- net DTR/RTS1: now also C1.2, JP1.3; no longer C2.2, JP7.3
- net GND: now also JP1.4, U$3.2; no longer JP1.5, JP1.6, JP2.5, JP2.6, JP3.5, JP3.6, JP4.5, JP4.6, JP5.5, JP5.6, JP6.5, JP6.6, JP7.4, U$2.2, U$2.3
- net RESET: now also C1.1; no longer C2.1
- net VCC: now also U$3.1; no longer U$2.1
Other:
- moved on the sheet: IC4, Q2, R2, R3, Y2
